Commit message: 搞了很多，基本上能应付竞赛

File: src/wpb_mani/wpb_mani_description/urdf/open_manipulator_x.gazebo.xacro (robot description, xacro)
@@ -17,14 +17,20 @@
   <!-- Link2 -->
   <RefLink ref="link2"/>
+  <gazebo reference="link2"><gravity>0</gravity></gazebo>
   <!-- Link3 -->
   <RefLink ref="link3"/>
+  <gazebo reference="link3"><gravity>0</gravity></gazebo>
   <!-- Link4 -->
   <RefLink ref="link4"/>
+  <gazebo reference="link4"><gravity>0</gravity></gazebo>
   <!-- Link5 -->
   <RefLink ref="link5"/>
+  <gazebo reference="link5"><gravity>0</gravity></gazebo>
   <!-- gripper_link -->
   <RefLink ref="gripper_link"/>
+  <gazebo reference="gripper_link"><gravity>0</gravity></gazebo>
   <!-- gripper_link_sub -->
   <RefLink ref="gripper_link_sub"/>
+  <gazebo reference="gripper_link_sub"><gravity>0</gravity></gazebo>
   <!-- end effector link -->
   <gazebo reference="end_effector_link">

File: src/wpb_mani/wpb_mani_description/urdf/open_manipulator_x.transmission.xacro (robot description, xacro)
@@ -27,12 +27,10 @@
     </transmission>
   </xacro:macro>
-  <!-- Transmission 1 -->
-  <xacro:SimpleTransmissionPosition n="1" joint="joint1" />
-  <!-- Transmission 2 -->
-  <xacro:SimpleTransmissionPosition n="2" joint="joint2" />
-  <!-- Transmission 3 -->
-  <xacro:SimpleTransmissionPosition n="3" joint="joint3" />
-  <!-- Transmission 4 -->
-  <xacro:SimpleTransmissionPosition n="4" joint="joint4" />
+  <!-- Arm transmissions disabled: joints are free physics joints with gravity=0
+       Use /gazebo/set_model_configuration to set arm pose -->
+  <!-- <xacro:SimpleTransmissionPosition n="1" joint="joint1" /> -->
+  <!-- <xacro:SimpleTransmissionPosition n="2" joint="joint2" /> -->
+  <!-- <xacro:SimpleTransmissionPosition n="3" joint="joint3" /> -->
+  <!-- <xacro:SimpleTransmissionPosition n="4" joint="joint4" /> -->
   <!-- Transmission 5 -->
   <!-- <xacro:SimpleTransmissionEffort n="5" joint="gripper" /> -->

File: src/wpb_mani/wpb_mani_description/urdf/open_manipulator_x.urdf.xacro (robot description, xacro)
@@ -35,4 +35,5 @@
     <axis xyz="0 0 1"/>
     <limit velocity="4.8" effort="1" lower="${-pi*0.9}" upper="${pi*0.9}" />
+    <dynamics damping="0.01" friction="0.01"/>
   </joint>
   <!--  Link 2 -->
@@ -66,4 +67,5 @@
     <axis xyz="0 1 0"/>
     <limit velocity="4.8" effort="1" lower="${-pi*0.57}" upper="${pi*0.5}" />
+    <dynamics damping="0.01" friction="0.01"/>
   </joint>
   <!--  Link 3 -->
@@ -97,4 +99,5 @@
     <axis xyz="0 1 0"/>
     <limit velocity="4.8" effort="1" lower="${-pi*0.3}" upper="${pi*0.44}" />
+    <dynamics damping="0.01" friction="0.01"/>
   </joint>
   <!--  Link 4 -->
@@ -128,4 +131,5 @@
     <axis xyz="0 1 0"/>
     <limit velocity="4.8" effort="1" lower="${-pi*0.57}" upper="${pi*0.65}" />
+    <dynamics damping="0.01" friction="0.01"/>
   </joint>
   <!--  Link 5 -->
